File: tp2/kicassv2/kicassv2.kicad_sch (KiCad schematic)
At the start: 28 parts, among them J1 CON_DATA, J2 CON_GND, J3 CON_Vcc, Q1 BC327, Q2 BC327, Q3 BC327, Q4 BC327

Commit message: commit pos-entrega
Connections:
- net Vcc: no longer U_DECO1.10 (2Y2), U_DECO1.12 (2Y0), U_DECO1.9 (2Y3)
- no-connect marks 10 -> 13
Changed lines of the file:
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@@
-	)
-	(junction
-		(at 262.89 143.51)
-		(diameter 0)
-		(color 0 0 0 0)
 	)
 	(junction
@@
 		(color 0 0 0 0)
 	)
-	(junction
-		(at 262.89 146.05)
-		(diameter 0)
-		(color 0 0 0 0)
-	)
 	(no_connect
 		(at 267.97 81.28)
@@
 	)
 	(no_connect
+		(at 262.89 146.05)
+	)
+	(no_connect
+		(at 262.89 140.97)
+	)
+	(no_connect
 		(at 232.41 83.82)
 	)
@@
 	)
 	(no_connect
+		(at 262.89 148.59)
+	)
+	(no_connect
 		(at 267.97 86.36)
 	)
@@
 	(wire
 		(pts
-			(xy 262.89 140.97) (xy 262.89 143.51)
-		)
-		(stroke
-			(width 0)
-			(type default)
-		)
-	)
-	(wire
-		(pts
 			(xy 143.51 60.96) (xy 143.51 73.66)
 		)
@@
 	(wire
 		(pts
-			(xy 262.89 143.51) (xy 262.89 146.05)
-		)
-		(stroke
-			(width 0)
-			(type default)
-		)
-	)
-	(wire
-		(pts
 			(xy 68.58 168.91) (xy 74.93 168.91)
 		)
@@
 		)
 		(stroke
-			(width 0)
-			(type default)
-		)
-	)
-	(wire
-		(pts
-			(xy 262.89 146.05) (xy 262.89 148.59)
-		)
-		(stroke
